File: hardware-libs/can.kicad_sch (KiCad schematic)
At the start: 10 parts, among them U1 TCAN332

Commit message: cambiado esquematico del can + tachadas un par de tareas
Parts:
- added C5: 100n, Capacitor_SMD:C_0603_1608Metric, symbol Device:C_Small
- U1: value TCAN332 -> TCAN3403DR-Q1
Connections:
- net +3.3V: now also U1.5 (SHDNVIO), C5.1
- net GND: now also U1.8 (STB), C5.2

Commit message: Update hardware libs to remove anotations + ticked some todos
Parts:
- renumbered C1 to C17, C3 to C18, C4 to C22, C2 to C9, C5 to C?, D1 to D2, JP1 to JP2, U1 to U5
Changed lines of the file:
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@@
 		(in_pos_files yes)
 		(dnp no)
-		(property "Reference" "#PWR05"
+		(property "Reference" "#PWR?"
 			(at 160.02 87.63 0)
 			(hide yes)
@@
 			(project "can"
 				(path "/6d6dd777-1a9f-4fc2-8a11-fafd679570cf"
-					(reference "#PWR05")
+					(reference "#PWR?")
 					(unit 1)
 				)
@@
 		(dnp no)
 		(fields_autoplaced yes)
-		(property "Reference" "JP1"
+		(property "Reference" "JP?"
 			(at 180.34 86.36 90)
 			(show_name no)
@@
 			(project "can"
 				(path "/6d6dd777-1a9f-4fc2-8a11-fafd679570cf"
-					(reference "JP1")
+					(reference "JP?")
 					(unit 1)
 				)
@@
 		(dnp no)
 		(fields_autoplaced yes)
-		(property "Reference" "#PWR04"
+		(property "Reference" "#PWR?"
 			(at 133.35 88.9 0)
 			(hide yes)
@@
 			(project "can"
 				(path "/6d6dd777-1a9f-4fc2-8a11-fafd679570cf"
-					(reference "#PWR04")
+					(reference "#PWR?")
 					(unit 1)
 				)
@@
 		(dnp no)
 		(fields_autoplaced yes)
-		(property "Reference" "FL1"
+		(property "Reference" "FL?"
 			(at 148.59 80.01 0)
 			(show_name no)
@@
 			(project "can"
 				(path "/6d6dd777-1a9f-4fc2-8a11-fafd679570cf"
-					(reference "FL1")
+					(reference "FL?")
 					(unit 1)
 				)
@@
 		(dnp no)
 		(fields_autoplaced yes)
-		(property "Reference" "#PWR02"
+		(property "Reference" "#PWR?"
 			(at 93.98 80.01 0)
 			(hide yes)
@@
 			(project "can"
 				(path "/6d6dd777-1a9f-4fc2-8a11-fafd679570cf"
-					(reference "#PWR02")
+					(reference "#PWR?")
 					(unit 1)
 				)
@@
 		(dnp no)
 		(fields_autoplaced yes)
-		(property "Reference" "C4"
+		(property "Reference" "C?"
 			(at 189.23 106.6799 0)
 			(show_name no)
@@
 			(project "can"
 				(path "/6d6dd777-1a9f-4fc2-8a11-fafd679570cf"
-					(reference "C4")
+					(reference "C?")
 					(unit 1)
 				)
@@
 		(dnp no)
 		(fields_autoplaced yes)
-		(property "Reference" "#PWR07"
+		(property "Reference" "#PWR?"
 			(at 185.42 118.11 0)
 			(hide yes)
@@
 			(project "can"
 				(path "/6d6dd777-1a9f-4fc2-8a11-fafd679570cf"
-					(reference "#PWR07")
+					(reference "#PWR?")
 					(unit 1)
 				)
@@
 		(dnp no)
 		(fields_autoplaced yes)
-		(property "Reference" "#PWR08"
+		(property "Reference" "#PWR?"
 			(at 74.93 93.98 0)
 			(hide yes)
@@
 			(project "can"
 				(path "/6d6dd777-1a9f-4fc2-8a11-fafd679570cf"
-					(reference "#PWR08")
+					(reference "#PWR?")
 					(unit 1)
 				)
@@
 		(dnp no)
 		(fields_autoplaced yes)
-		(property "Reference" "C3"
+		(property "Reference" "C?"
 			(at 189.23 68.5799 0)
 			(show_name no)
@@
 			(project "can"
 				(path "/6d6dd777-1a9f-4fc2-8a11-fafd679570cf"
-					(reference "C3")
+					(reference "C?")
 					(unit 1)
 				)
@@
 		(dnp no)
 		(fields_autoplaced yes)
-		(property "Reference" "R1"
+		(property "Reference" "R?"
 			(at 187.96 77.4699 0)
 			(show_name no)
@@
 			(project "can"
 				(path "/6d6dd777-1a9f-4fc2-8a11-fafd679570cf"
-					(reference "R1")
+					(reference "R?")
 					(unit 1)
 				)
@@
 		(dnp no)
 		(fields_autoplaced yes)
-		(property "Reference" "C5"
+		(property "Reference" "C?"
 			(at 63.5 93.9799 0)
 			(show_name no)
@@
 			(project "can"
 				(path "/6d6dd777-1a9f-4fc2-8a11-fafd679570cf"
-					(reference "C5")
+					(reference "C?")
 					(unit 1)
 				)
@@
 		(dnp no)
 		(fields_autoplaced yes)
-		(property "Reference" "#PWR03"
+		(property "Reference" "#PWR?"
 			(at 93.98 106.68 0)
 			(hide yes)
@@
 			(project "can"
 				(path "/6d6dd777-1a9f-4fc2-8a11-fafd679570cf"
-					(reference "#PWR03")
+					(reference "#PWR?")
 					(unit 1)
 				)
@@
 		(dnp no)
 		(fields_autoplaced yes)
-		(property "Reference" "#PWR09"
+		(property "Reference" "#PWR?"
 			(at 60.96 93.98 0)
 			(hide yes)
@@
 			(project "can"
 				(path "/6d6dd777-1a9f-4fc2-8a11-fafd679570cf"
-					(reference "#PWR09")
+					(reference "#PWR?")
 					(unit 1)
 				)
@@
 		(in_pos_files yes)
 		(dnp no)
-		(property "Reference" "C2"
+		(property "Reference" "C?"
 			(at 170.18 80.01 90)
 			(show_name no)
@@
 			(project "can"
 				(path "/6d6dd777-1a9f-4fc2-8a11-fafd679570cf"
-					(reference "C2")
+					(reference "C?")
 					(unit 1)
 				)
@@
 		(in_pos_files yes)
 		(dnp no)
-		(property "Reference" "D1"
+		(property "Reference" "D?"
 			(at 127.508 85.344 90)
 			(show_name no)
@@
 			(project "can"
 				(path "/6d6dd777-1a9f-4fc2-8a11-fafd679570cf"
-					(reference "D1")
+					(reference "D?")
 					(unit 1)
 				)
@@
 		(dnp no)
 		(fields_autoplaced yes)
-		(property "Reference" "C1"
+		(property "Reference" "C?"
 			(at 87.6363 69.85 90)
 			(show_name no)
@@
 			(project "can"
 				(path "/6d6dd777-1a9f-4fc2-8a11-fafd679570cf"
-					(reference "C1")
+					(reference "C?")
 					(unit 1)
 				)
@@
 		(dnp no)
 		(fields_autoplaced yes)
-		(property "Reference" "#PWR01"
+		(property "Reference" "#PWR?"
 			(at 74.93 76.2 0)
 			(hide yes)
@@
 			(project "can"
 				(path "/6d6dd777-1a9f-4fc2-8a11-fafd679570cf"
-					(reference "#PWR01")
+					(reference "#PWR?")
 					(unit 1)
 				)
@@
 		(dnp no)
 		(fields_autoplaced yes)
-		(property "Reference" "#PWR06"
+		(property "Reference" "#PWR?"
 			(at 185.42 59.69 0)
 			(hide yes)
@@
 			(project "can"
 				(path "/6d6dd777-1a9f-4fc2-8a11-fafd679570cf"
-					(reference "#PWR06")
+					(reference "#PWR?")
 					(unit 1)
 				)
@@
 		(dnp no)
 		(fields_autoplaced yes)
-		(property "Reference" "U1"
+		(property "Reference" "U?"
 			(at 96.1741 76.2 0)
 			(show_name no)
@@
 			(project "can"
 				(path "/6d6dd777-1a9f-4fc2-8a11-fafd679570cf"
-					(reference "U1")
+					(reference "U?")
 					(unit 1)
 				)
@@
 		(dnp no)
 		(fields_autoplaced yes)
-		(property "Reference" "R2"
+		(property "Reference" "R?"
 			(at 187.96 95.2499 0)
 			(show_name no)
@@
 			(project "can"
 				(path "/6d6dd777-1a9f-4fc2-8a11-fafd679570cf"
-					(reference "R2")
+					(reference "R?")
 					(unit 1)
 				)
@@
 		(dnp no)
 		(fields_autoplaced yes)
-		(property "Reference" "#PWR010"
+		(property "Reference" "#PWR?"
 			(at 60.96 104.14 0)
 			(hide yes)
@@
 			(project "can"
 				(path "/6d6dd777-1a9f-4fc2-8a11-fafd679570cf"
-					(reference "#PWR010")
-					(unit 1)
-				)
+					(reference "#PWR?")
+					(unit 1)
+				)
