File: hardware-libs/power.kicad_sch (KiCad schematic)
At the start: 8 parts, among them U1 TSR_1-2450, U2 LM1117MP-3.3

Commit message: Update hardware libs to remove anotations + ticked some todos
Parts:
- renumbered C3 to C?, C4 to C?, C1 to C?, C2 to C?, F1 to F?, L1 to L?, U2 to U?, U1 to U?
Changed lines of the file:
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@@
 		(dnp no)
 		(fields_autoplaced yes)
-		(property "Reference" "#PWR09"
+		(property "Reference" "#PWR?"
 			(at 160.02 45.72 0)
 			(hide yes)
@@
 			(project "power"
 				(path "/193dd9e0-5ae8-43aa-a6d1-cd57fa78b58f"
-					(reference "#PWR09")
+					(reference "#PWR?")
 					(unit 1)
 				)
@@
 		(in_pos_files yes)
 		(dnp no)
-		(property "Reference" "#FLG02"
+		(property "Reference" "#FLG?"
 			(at 18.415 55.88 0)
 			(hide yes)
@@
 			(project "power"
 				(path "/193dd9e0-5ae8-43aa-a6d1-cd57fa78b58f"
-					(reference "#FLG02")
+					(reference "#FLG?")
 					(unit 1)
 				)
@@
 		(dnp no)
 		(fields_autoplaced yes)
-		(property "Reference" "#PWR02"
+		(property "Reference" "#PWR?"
 			(at 26.67 55.88 0)
 			(hide yes)
@@
 			(project "power"
 				(path "/193dd9e0-5ae8-43aa-a6d1-cd57fa78b58f"
-					(reference "#PWR02")
+					(reference "#PWR?")
 					(unit 1)
 				)
@@
 		(dnp no)
 		(fields_autoplaced yes)
-		(property "Reference" "C3"
+		(property "Reference" "C?"
 			(at 149.86 33.02 0)
 			(show_name no)
@@
 			(project "power"
 				(path "/193dd9e0-5ae8-43aa-a6d1-cd57fa78b58f"
-					(reference "C3")
+					(reference "C?")
 					(unit 1)
 				)
@@
 		(dnp no)
 		(fields_autoplaced yes)
-		(property "Reference" "C4"
+		(property "Reference" "C?"
 			(at 176.53 33.02 0)
 			(show_name no)
@@
 			(project "power"
 				(path "/193dd9e0-5ae8-43aa-a6d1-cd57fa78b58f"
-					(reference "C4")
+					(reference "C?")
 					(unit 1)
 				)
@@
 		(dnp no)
 		(fields_autoplaced yes)
-		(property "Reference" "#PWR04"
+		(property "Reference" "#PWR?"
 			(at 46.99 52.07 0)
 			(hide yes)
@@
 			(project "power"
 				(path "/193dd9e0-5ae8-43aa-a6d1-cd57fa78b58f"
-					(reference "#PWR04")
+					(reference "#PWR?")
 					(unit 1)
 				)
@@
 		(dnp no)
 		(fields_autoplaced yes)
-		(property "Reference" "C1"
+		(property "Reference" "C?"
 			(at 50.8 36.83 0)
 			(show_name no)
@@
 			(project "power"
 				(path "/193dd9e0-5ae8-43aa-a6d1-cd57fa78b58f"
-					(reference "C1")
+					(reference "C?")
 					(unit 1)
 				)
@@
 		(dnp no)
 		(fields_autoplaced yes)
-		(property "Reference" "F1"
+		(property "Reference" "F?"
 			(at 34.29 29.21 90)
 			(show_name no)
@@
 			(project "power"
 				(path "/193dd9e0-5ae8-43aa-a6d1-cd57fa78b58f"
-					(reference "F1")
+					(reference "F?")
 					(unit 1)
 				)
@@
 		(in_pos_files yes)
 		(dnp no)
-		(property "Reference" "#FLG03"
+		(property "Reference" "#FLG?"
 			(at 69.85 32.385 0)
 			(hide yes)
@@
 			(project "power"
 				(path "/193dd9e0-5ae8-43aa-a6d1-cd57fa78b58f"
-					(reference "#FLG03")
+					(reference "#FLG?")
 					(unit 1)
 				)
@@
 		(dnp no)
 		(fields_autoplaced yes)
-		(property "Reference" "#PWR010"
+		(property "Reference" "#PWR?"
 			(at 181.61 31.75 0)
 			(hide yes)
@@
 			(project "power"
 				(path "/193dd9e0-5ae8-43aa-a6d1-cd57fa78b58f"
-					(reference "#PWR010")
+					(reference "#PWR?")
 					(unit 1)
 				)
@@
 		(dnp no)
 		(fields_autoplaced yes)
-		(property "Reference" "#PWR06"
+		(property "Reference" "#PWR?"
 			(at 83.82 53.34 0)
 			(hide yes)
@@
 			(project "power"
 				(path "/193dd9e0-5ae8-43aa-a6d1-cd57fa78b58f"
-					(reference "#PWR06")
+					(reference "#PWR?")
 					(unit 1)
 				)
@@
 		(dnp no)
 		(fields_autoplaced yes)
-		(property "Reference" "C2"
+		(property "Reference" "C?"
 			(at 68.58 36.83 0)
 			(show_name no)
@@
 			(project "power"
 				(path "/193dd9e0-5ae8-43aa-a6d1-cd57fa78b58f"
-					(reference "C2")
+					(reference "C?")
 					(unit 1)
 				)
@@
 		(dnp no)
 		(fields_autoplaced yes)
-		(property "Reference" "#PWR07"
+		(property "Reference" "#PWR?"
 			(at 116.84 36.83 0)
 			(hide yes)
@@
 			(project "power"
 				(path "/193dd9e0-5ae8-43aa-a6d1-cd57fa78b58f"
-					(reference "#PWR07")
+					(reference "#PWR?")
 					(unit 1)
 				)
@@
 		(in_pos_files yes)
 		(dnp no)
-		(property "Reference" "U2"
+		(property "Reference" "U?"
 			(at 160.02 22.86 0)
 			(show_name no)
@@
 			(project "power"
 				(path "/193dd9e0-5ae8-43aa-a6d1-cd57fa78b58f"
-					(reference "U2")
+					(reference "U?")
 					(unit 1)
 				)
@@
 		(dnp no)
 		(fields_autoplaced yes)
-		(property "Reference" "#PWR08"
+		(property "Reference" "#PWR?"
 			(at 133.35 31.75 0)
 			(hide yes)
@@
 			(project "power"
 				(path "/193dd9e0-5ae8-43aa-a6d1-cd57fa78b58f"
-					(reference "#PWR08")
+					(reference "#PWR?")
 					(unit 1)
 				)
@@
 		(dnp no)
 		(fields_autoplaced yes)
-		(property "Reference" "#PWR03"
+		(property "Reference" "#PWR?"
 			(at 27.94 31.75 0)
 			(hide yes)
@@
 			(project "power"
 				(path "/193dd9e0-5ae8-43aa-a6d1-cd57fa78b58f"
-					(reference "#PWR03")
+					(reference "#PWR?")
 					(unit 1)
 				)
@@
 		(in_pos_files yes)
 		(dnp no)
-		(property "Reference" "#FLG01"
+		(property "Reference" "#FLG?"
 			(at 18.415 49.53 0)
 			(hide yes)
@@
 			(project "power"
 				(path "/193dd9e0-5ae8-43aa-a6d1-cd57fa78b58f"
-					(reference "#FLG01")
+					(reference "#FLG?")
 					(unit 1)
 				)
@@
 		(dnp no)
 		(fields_autoplaced yes)
-		(property "Reference" "L1"
+		(property "Reference" "L?"
 			(at 55.88 26.67 0)
 			(show_name no)
@@
 			(project "power"
 				(path "/193dd9e0-5ae8-43aa-a6d1-cd57fa78b58f"
-					(reference "L1")
+					(reference "L?")
 					(unit 1)
 				)
@@
 		(dnp no)
 		(fields_autoplaced yes)
-		(property "Reference" "#PWR01"
+		(property "Reference" "#PWR?"
 			(at 16.51 49.53 0)
 			(hide yes)
@@
 			(project "power"
 				(path "/193dd9e0-5ae8-43aa-a6d1-cd57fa78b58f"
-					(reference "#PWR01")
+					(reference "#PWR?")
 					(unit 1)
 				)
@@
 		(dnp no)
 		(fields_autoplaced yes)
-		(property "Reference" "U1"
+		(property "Reference" "U?"
 			(at 83.82 27.94 0)
 			(show_name no)
@@
 			(project "power"
 				(path "/193dd9e0-5ae8-43aa-a6d1-cd57fa78b58f"
-					(reference "U1")
+					(reference "U?")
 					(unit 1)
 				)
@@
 		(dnp no)
 		(fields_autoplaced yes)
-		(property "Reference" "#PWR05"
+		(property "Reference" "#PWR?"
 			(at 64.77 52.07 0)
 			(hide yes)
@@
 			(project "power"
 				(path "/193dd9e0-5ae8-43aa-a6d1-cd57fa78b58f"
-					(reference "#PWR05")
-					(unit 1)
-				)
+					(reference "#PWR?")
+					(unit 1)
+				)
