File: hardware-libs/stm32f1_core.kicad_sch (KiCad schematic)
At the start: 22 parts, among them J1 DEBUG, SW1 RST, U1 STM32F103C8Tx, Y1 8mHz

Commit message: Update hardware libs to remove anotations + ticked some todos
Parts:
- renumbered C2 to C1, C4 to C1, C7 to C14, C3 to C15, C9 to C16, C6 to C2, C8 to C3, C11 to C4, C1 to C5, C10 to C9, R1 to R4, R3 to R6, R2 to R7, R4 to R7, R5 to R8, R6 to R9
